File: hoja-dongle.kicad_sch (KiCad schematic)
At the start: 64 parts, among them J2 USB4080-03-A_REVA1, J3 Conn_01x04_Pin, P1 RPI-RM2, Q1 BSS138DW, Q2 BSS138DW, SW1 1TS026A-1000-0550, SW2 SW_Push, SW3 SW_Push, U1 USBLC6-2P6, U2 USBLC6-2P6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

Commit message: prod
Parts:
- added R13: 51K, Resistor_SMD:R_0201_0603Metric, symbol Device:R
- J2: Link (none) -> https://www.digikey.com/en/products/detail/gct/USB4080-03-A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; MPN (none) -> USB4080-03-A
- R11: Link (none) -> https://www.lcsc.com/product-detail/Chip-Resistor-Surface-M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
- R19, R20, R21: value 100R -> 27R; LCSC C77623 -> C273268; MPN RC0201FR-07100RL -> RC0201FR-0727RL
- U1, U2, U3: LCSC (none) -> C15999; Link (none) -> https://www.lcsc.com/product-detail/C15999.html?s_z=n_USBLC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; MPN (none) -> USBLC6-2P6; Package (none) -> SOT-666-6
Connections:
- net +3V3_PRE: now also R13.2
- net GND: now also R13.1
